Commit message: Made the top part of the lift mechanism mimic the bottom part to emulate a parallelogram

File: rose21_urdf/rose21.xacro (robot description, xacro)
@@ -137,6 +137,5 @@
       <axis xyz="0 1 0" />
       <origin xyz="${-liftsides_size_x} 0 0" rpy="0 0 0"/>
-      <dynamics damping="1.0" friction="1.0"/>
-      <limit effort="10.0" lower="0" upper="0" velocity="1.0"/>
+      <mimic joint="lift_mid_bottom_joint" multiplier="-1"/>
     </joint>
   </xacro:macro>

Commit message: Reintroduced the two lift beams as well

File: rose21_urdf/rose21.xacro (robot description, xacro)
@@ -91,5 +91,4 @@
   </link>
   <!-- joint between base and lift_left -->
-  <!-- URDF DOES NOT SUPPORT JOINT LOOPS SO ONLY USE ONE BAR OF THE LIFFT FOR NOW
   <joint name="lift_left_bottom_joint" type="revolute">
     <parent link="base_link"/>
@@ -97,11 +96,8 @@
     <axis xyz="0 1 0" />
     <origin xyz="${base_size_x/2 - 0.055 - 0.14} ${liftsides_pose_y} ${base_pose_z}" rpy="0 0 0"/>
-    <dynamics damping="1.0" friction="1.0"/>
+    <mimic joint="lift_mid_bottom_joint"/>
     <limit effort="10.0" lower="0.0" upper="${pi/2}" velocity="1.0"/>
   </joint>
-  -->
-  <!-- lift left -->
-  <!-- URDF DOES NOT SUPPORT JOINT LOOPS SO ONLY USE ONE BAR OF THE LIFFT FOR NOW
-  <link name='lift_left'>
+  <!-- lift left -->  <link name='lift_left'>
     <xacro:default_box  xyz=  "${-liftsides_size_x/2} 0 0"
                         rpy=  "0 0 0"
@@ -109,7 +105,5 @@
     <xacro:default_inertial mass="0.5"/>
   </link>
-  -->
   <!-- joint between base and lift_right -->
-  <!-- URDF DOES NOT SUPPORT JOINT LOOPS SO ONLY USE ONE BAR OF THE LIFFT FOR NOW
   <joint name="lift_right_bottom_joint" type="revolute">
     <parent link="base_link"/>
@@ -117,10 +111,8 @@
     <axis xyz="0 1 0" />
     <origin xyz="${base_size_x/2 - 0.055 - 0.14} ${-liftsides_pose_y} ${base_pose_z}" rpy="0 0 0"/>
-    <dynamics damping="1.0" friction="1.0"/>
     <limit effort="10.0" lower="0.0" upper="${pi/2}" velocity="1.0"/>
-  </joint>
-  -->
+    <mimic joint="lift_mid_bottom_joint"/>
+  </joint>
   <!-- lift right -->
-  <!-- URDF DOES NOT SUPPORT JOINT LOOPS SO ONLY USE ONE BAR OF THE LIFFT FOR NOW
   <link name='lift_right'>
       <xacro:default_box xyz=  "${-liftsides_size_x/2} 0 0"
@@ -129,5 +121,4 @@
      <xacro:default_inertial mass="0.5"/>
   </link>
-  -->
   <!-- macro for joining the lift bars to the top of rose -->
   <xacro:macro name="lift_bar_joint" params="parent">

Commit message: Reordered neck joints and links to accomodate for longer neck. Joint order is OK now, dimensions not yet

File: rose21_urdf/rose21.xacro (robot description, xacro)
@@ -31,12 +31,17 @@
   <xacro:property name="lifttopbox_size_x" value="0.29" />
   <xacro:property name="lifttopbox_size_y" value="0.24" />
-  <xacro:property name="lifttopbox_size_z" value="0.57" />
+  <xacro:property name="lifttopbox_size_z" value="0.697" /> <!--This includes the shoulders -->
   <xacro:property name="lifttopbox_pose_x" value="0.0" />
   <xacro:property name="lifttopbox_pose_y" value="0.0" />
   <xacro:property name="lifttopbox_pose_z" value="0.285"/>
+  <xacro:property name="shoulders_size_x" value="0.265" />
+  <xacro:property name="shoulders_size_y" value="0.58" />
+  <xacro:property name="shoulders_size_z" value="0.177" /> <!--This includes the shoulders -->
   <xacro:property name="lift_rpy" value="0 0 0"/>
-  <xacro:property name="neck_pan_size_x" value="0.05" />
-  <xacro:property name="neck_pan_size_y" value="0.03" />
-  <xacro:property name="neck_pan_size_z" value="0.04" />
+  <xacro:property name="neck_tube_size_z" value="0.07" />
+  <xacro:property name="neck_tube_diameter" value="0.03" />
+  <xacro:property name="neck_pan_size_x" value="0.298" />
+  <xacro:property name="neck_pan_size_y" value="0.04" />
+  <xacro:property name="neck_pan_size_z" value="0.02" />
   <xacro:property name="neck_pan_pose_x" value="0.015" />
   <xacro:property name="neck_pan_pose_y" value="0.00" />
@@ -45,7 +50,7 @@
   <xacro:property name="neck_tilt_size_y" value="0.04" />
   <xacro:property name="neck_tilt_size_z" value="0.055" />
-  <xacro:property name="neck_tilt_pose_x" value="0.00" />
+  <xacro:property name="neck_tilt_pose_x" value="0.28" /> <!--Distance between tilt axis and neck pan tube -->
   <xacro:property name="neck_tilt_pose_y" value="0.00" />
-  <xacro:property name="neck_tilt_pose_z" value="0.05" />
+  <xacro:property name="neck_tilt_pose_z" value="0.115" /> <!--Height of the tilt axis from top of shoulders-->
   <xacro:property name="kinect_size_x" value="0.073" />
   <xacro:property name="kinect_size_y" value="0.270" />
@@ -167,25 +172,30 @@
   <!-- START neck -->
   <!-- joint between lift_link and neck_pan -->
-  <joint name="neck_fixed_joint" type="fixed">
+  <joint name="neck_pan_joint" type="revolute">
     <parent link="lift_link"/>
     <child link="neck_pan"/>
-    <axis xyz="0 1 0" />
-    <origin xyz="0 0 ${lifttopbox_size_z}" rpy="0 0 0"/>
-  </joint>
-  <!-- neck_pan -->
+    <axis xyz="0 0 1" />
+    <origin xyz="0 0 ${lifttopbox_size_z + shoulders_size_z}" rpy="0 0 0"/>
+    <dynamics damping="1.0" friction="1.0"/>
+    <limit effort="1.0" lower="-0.7853" upper="0.7853" velocity="10.0"/>
+  </joint>
+  <!-- neck_pan is the tube and bar that rotate to pan the kinect around that looks like:
+   ______#          with the # being the motor-part of the tilt-servo
+  |
+   -->
   <link name='neck_pan'>
-    <xacro:default_box  xyz=  "0 0 ${neck_pan_size_z/2}"
+    <xacro:default_box  xyz=  "${neck_pan_size_x /2} 0 ${neck_pan_size_z/2}"
                         rpy=  "0 0 0"
                         size= "${neck_pan_size_x} ${neck_pan_size_y} ${neck_pan_size_z}"/>
     <xacro:default_inertial mass="0.25"/>
   </link>
-  <!-- joint between neck_pan and neck_tilt -->
-  <joint name="neck_pan_joint" type="revolute">
+   <!-- joint between neck_pan and neck_tilt-->
+  <joint name="neck_tilt_joint" type="revolute">
     <parent link="neck_pan"/>
     <child link="neck_tilt"/>
-    <axis xyz="0 0 1" />
-    <origin xyz="${neck_pan_pose_x} 0 ${neck_pan_size_z}" rpy="0 0 0"/>
+    <axis xyz="0 1 0" />
+    <origin xyz="${neck_tilt_pose_x} ${neck_tilt_pose_y} ${neck_tilt_pose_z}" rpy="0 0 0"/>
     <dynamics damping="1.0" friction="1.0"/>
-    <limit effort="1.0" lower="-0.7853" upper="0.7853" velocity="10.0"/>
+    <limit effort="1.0" lower="-1.5707" upper="1.5707" velocity="1.0"/>
   </joint>
   <!-- neck_tilt -->
@@ -196,12 +206,10 @@
     <xacro:default_inertial mass="0.25"/>
   </link>
-   <!-- joint between neck_tilt and kinect -->
-  <joint name="neck_tilt_joint" type="revolute">
+  <!-- joint between neck_tilt and kinect-->
+  <joint name="kinect_fiz" type="fixed">
     <parent link="neck_tilt"/>
     <child link="kinect"/>
     <axis xyz="0 1 0" />
     <origin xyz="${kinect_pose_x} ${kinect_pose_y} ${kinect_pose_z}" rpy="0 0 0"/>
-    <dynamics damping="1.0" friction="1.0"/>
-    <limit effort="1.0" lower="-1.5707" upper="1.5707" velocity="1.0"/>
   </joint>
   <!-- END neck -->

Commit message: Put neck-pan in middle of lift-top-box

File: rose21_urdf/rose21.xacro (robot description, xacro)
@@ -31,11 +31,11 @@
   <xacro:property name="lifttopbox_size_x" value="0.29" />
   <xacro:property name="lifttopbox_size_y" value="0.24" />
-  <xacro:property name="lifttopbox_size_z" value="0.697" /> <!--This includes the shoulders -->
-  <xacro:property name="lifttopbox_pose_x" value="0.0" />
+  <xacro:property name="lifttopbox_size_z" value="0.48" /> <!--This excludes the shoulders -->
+  <xacro:property name="lifttopbox_pose_x" value="-0.10" />
   <xacro:property name="lifttopbox_pose_y" value="0.0" />
   <xacro:property name="lifttopbox_pose_z" value="0.285"/>
   <xacro:property name="shoulders_size_x" value="0.265" />
   <xacro:property name="shoulders_size_y" value="0.58" />
-  <xacro:property name="shoulders_size_z" value="0.177" /> <!--This includes the shoulders -->
+  <xacro:property name="shoulders_size_z" value="0.177" />
   <xacro:property name="lift_rpy" value="0 0 0"/>
   <xacro:property name="neck_tube_size_z" value="0.07" />
@@ -138,5 +138,5 @@
   <!-- lift top box -->
   <link name='lift_link'>
-    <xacro:default_box  xyz=  "-0.10 0 ${lifttopbox_size_z/2}"
+    <xacro:default_box  xyz=  "${lifttopbox_pose_x} 0 ${lifttopbox_size_z/2}"
                         rpy=  "0 0 0"
                         size= "${lifttopbox_size_x} ${lifttopbox_size_y} ${lifttopbox_size_z}"/>
@@ -176,5 +176,5 @@
     <child link="neck_pan"/>
     <axis xyz="0 0 1" />
-    <origin xyz="0 0 ${lifttopbox_size_z + shoulders_size_z}" rpy="0 0 0"/>
+    <origin xyz="${lifttopbox_pose_x} 0 ${lifttopbox_size_z + shoulders_size_z}" rpy="0 0 0"/>
     <dynamics damping="1.0" friction="1.0"/>
     <limit effort="1.0" lower="-0.7853" upper="0.7853" velocity="10.0"/>
@@ -185,5 +185,5 @@
    -->
   <link name='neck_pan'>
-    <xacro:default_box  xyz=  "${neck_pan_size_x /2} 0 ${neck_pan_size_z/2}"
+    <xacro:default_box  xyz=  "${neck_pan_size_x/2} 0 ${neck_pan_size_z/2 + neck_tube_size_z}"
                         rpy=  "0 0 0"
                         size= "${neck_pan_size_x} ${neck_pan_size_y} ${neck_pan_size_z}"/>
@@ -207,5 +207,5 @@
   </link>
   <!-- joint between neck_tilt and kinect-->
-  <joint name="kinect_fiz" type="fixed">
+  <joint name="kinect_fix" type="fixed">
     <parent link="neck_tilt"/>
     <child link="kinect"/>

Commit message: Neck tilt works, only the servo itself tilts but the camera works

File: rose21_urdf/rose21.xacro (robot description, xacro)
@@ -48,6 +48,7 @@
   <xacro:property name="neck_pan_pose_z" value="0.00" />
   <xacro:property name="neck_tilt_size_x" value="0.033" />
-  <xacro:property name="neck_tilt_size_y" value="0.04" />
-  <xacro:property name="neck_tilt_size_z" value="0.055" />
+  <xacro:property name="neck_tilt_size_y" value="0.035" />
+  <xacro:property name="neck_tilt_size_z" value="0.048" />
+  <xacro:property name="neck_tilt_servo_center_z" value="0.033" />
   <xacro:property name="neck_tilt_pose_x" value="0.28" /> <!--Distance between tilt axis and neck pan tube -->
   <xacro:property name="neck_tilt_pose_y" value="0.00" />
@@ -201,5 +202,5 @@
   <!-- neck_tilt -->
   <link name='neck_tilt'>
-    <xacro:default_box  xyz=  "0 0 ${neck_tilt_size_z/2}"
+    <xacro:default_box  xyz=  "0 0 ${neck_tilt_size_z/2 - neck_tilt_servo_center_z}"
                         rpy=  "0 0 0"
                         size= "${neck_tilt_size_x} ${neck_tilt_size_y} ${neck_tilt_size_z}"/>

Commit message: Add the links/frames of the camera to urdf

File: rose21_urdf/rose21.xacro (robot description, xacro)
@@ -266,4 +266,64 @@
     <plugin name="NeckController" filename="libNeckController.so"/>
   </gazebo>
+  <joint name="link2" type="fixed">
+      <parent link="neck_tilt"/>
+      <child link="camera_center_link"/>
+    </joint>
+    <link name="camera_center_link">
+      <visual>
+        <origin xyz="0 0 0" rpy="0 0 0" />
+        <geometry>
+          <box size="0 0 0" />
+        </geometry>
+        <material name="black">
+          <color rgba=".1 .1 .1 1" />
+        </material>
+      </visual>
+    </link>
+    <joint name="link3" type="fixed">
+      <parent link="camera_center_link"/>
+      <child link="camera_link"/>
+    </joint>
+    <link name="camera_link">
+      <visual>
+        <origin xyz="0 0 0" rpy="0 0 0" />
+        <geometry>
+          <box size="0.06 0.28 0.04" />
+        </geometry>
+        <material name="black">
+          <color rgba=".1 .1 .1 1" />
+        </material>
+      </visual>
+    </link>
+    <joint name="link4" type="fixed">
+      <parent link="camera_link"/>
+      <child link="camera_rgb_frame"/>
+    </joint>
+    <link name="camera_rgb_frame">
+      <visual>
+        <origin xyz="0 0 0" rpy="0 0 0" />
+        <geometry>
+          <box size="0 0 0" />
+        </geometry>
+        <material name="black">
+          <color rgba=".1 .1 .1 1" />
+        </material>
+      </visual>
+    </link>
+    <joint name="link5" type="fixed">
+      <parent link="camera_rgb_frame"/>
+      <child link="camera_rgb_optical_frame"/>
+    </joint>
+    <link name="camera_rgb_optical_frame">
+      <visual>
+        <origin xyz="0 0 0" rpy="0 0 0" />
+        <geometry>
+          <box size="0 0 0" />
+        </geometry>
+        <material name="black">
+          <color rgba=".1 .1 .1 1" />
+        </material>
+      </visual>
+    </link>
     <!-- START Hokuyo -->
   <joint name="hokuyo_joint" type="revolute">

Commit message: Using the robot+joint-state_publisher in the description. I noticed that the tilt joint in the neck is mirrored and should turn in the other direction

File: rose21_urdf/rose21.xacro (robot description, xacro)
@@ -173,5 +173,5 @@
   <!-- START neck -->
   <!-- joint between lift_link and neck_pan -->
-  <joint name="neck_pan_joint" type="revolute">
+  <joint name="pan_joint" type="revolute">
     <parent link="lift_link"/>
     <child link="neck_pan"/>
@@ -192,5 +192,5 @@
   </link>
    <!-- joint between neck_pan and neck_tilt-->
-  <joint name="neck_tilt_joint" type="revolute">
+  <joint name="tilt_joint" type="revolute">
     <parent link="neck_pan"/>
     <child link="neck_tilt"/>

Commit message: Axis of tilt_joint now rotates the other way which is consistent with reality

File: rose21_urdf/rose21.xacro (robot description, xacro)
@@ -195,5 +195,5 @@
     <parent link="neck_pan"/>
     <child link="neck_tilt"/>
-    <axis xyz="0 1 0" />
+    <axis xyz="0 -1 0" />
     <origin xyz="${neck_tilt_pose_x} ${neck_tilt_pose_y} ${neck_tilt_pose_z}" rpy="0 0 0"/>
     <dynamics damping="1.0" friction="1.0"/>

Commit message: Using copied-over meshes and xacro's so rose20_description in rose_simulator isn't needed

File: rose21_urdf/rose21.xacro (robot description, xacro)
@@ -1,5 +1,5 @@
 <robot name="Rose20" xmlns:xacro="http://www.ros.org/wiki/xacro">
-  <xacro:include filename="$(find rose20_description)/common.xacro" />
-  <xacro:include filename="$(find rose20_description)/wheel_unit_60mm/wheel_unit_60mm_macro.xacro" />
+  <xacro:include filename="$(find rose21_urdf)/common.xacro" />
+  <xacro:include filename="$(find rose21_urdf)/urdf/wheel_unit_60mm/wheel_unit_60mm_macro.xacro" />
   <xacro:property name="base_size_x" value="0.76" />
   <xacro:property name="base_size_y" value="0.58" />
@@ -223,5 +223,5 @@
       <origin xyz="0 0 0.036" rpy="0 0 0" />
         <geometry>
-          <mesh filename="package://rose20_description/rose20/meshes/kinect.dae"/>
+          <mesh filename="package://rose21_urdf/meshes/kinect.dae"/>
         </geometry>
     </visual>

Commit message: Added a base_link_extension link for testing purposes that willl be transformed into the 'bakje'

File: rose21_urdf/rose21.xacro (robot description, xacro)
@@ -75,4 +75,15 @@
     <xacro:default_inertial mass="30.0"/>
   </link>
+  <joint name="extension_joint" type="fixed">
+    <parent link="base_link"/>
+    <child link="base_link_extension"/>
+    <origin xyz="3 0 0" rpy="0 0 0"/>
+  </joint>
+  <link name='base_link_extension'>
+    <xacro:default_box  xyz=  "0 0 0"
+                        rpy=  "0 0 0"
+                        size= "${base_size_x} ${base_size_y} ${base_size_z}"/>
+    <xacro:default_inertial mass="30.0"/>
+  </link>
   <!-- Wheel units -->
   <xacro:wheel_unit_60mm name="FL" parent="base_link" xyz="${wheel_front_x} ${-wheelbase_width} ${base_pose_z - base_size_z/2}" rpy="0 0 ${-pi/2}"/>

Commit message: Added rose's tray properly

File: rose21_urdf/rose21.xacro (robot description, xacro)
@@ -8,4 +8,10 @@
   <xacro:property name="base_pose_y" value="0.0" />
   <xacro:property name="base_pose_z" value="0.20" />
+  <xacro:property name="tray_size_x" value="0.20" />
+  <xacro:property name="tray_size_y" value="0.20" />
+  <xacro:property name="tray_size_z" value="0.05" />
+  <xacro:property name="tray_pose_x" value="0.135" />
+  <xacro:property name="tray_pose_y" value="0.0" />
+  <xacro:property name="tray_pose_z" value="0.13" />
   <xacro:property name="wheel_front_x"    value="0.28" />
   <xacro:property name="wheel_back_x"     value="-0.305" />
@@ -75,15 +81,4 @@
     <xacro:default_inertial mass="30.0"/>
   </link>
-  <joint name="extension_joint" type="fixed">
-    <parent link="base_link"/>
-    <child link="base_link_extension"/>
-    <origin xyz="3 0 0" rpy="0 0 0"/>
-  </joint>
-  <link name='base_link_extension'>
-    <xacro:default_box  xyz=  "0 0 0"
-                        rpy=  "0 0 0"
-                        size= "${base_size_x} ${base_size_y} ${base_size_z}"/>
-    <xacro:default_inertial mass="30.0"/>
-  </link>
   <!-- Wheel units -->
   <xacro:wheel_unit_60mm name="FL" parent="base_link" xyz="${wheel_front_x} ${-wheelbase_width} ${base_pose_z - base_size_z/2}" rpy="0 0 ${-pi/2}"/>
@@ -182,4 +177,15 @@
     </plugin>
   </gazebo>
+  <joint name="tray_mount" type="fixed">
+    <parent link="lift_link"/>
+    <child link="tray"/>
+    <origin xyz="0 0 0" rpy="0 0 0"/>
+  </joint>
+  <link name='tray'>
+    <xacro:default_box  xyz=  "${tray_pose_x} ${tray_pose_y} ${tray_pose_z}"
+                        rpy=  "0 0 0"
+                        size= "${tray_size_x} ${tray_size_y} ${tray_size_z}"/>
+    <xacro:default_inertial mass="2.0"/>
+  </link>
   <!-- START neck -->
   <!-- joint between lift_link and neck_pan -->

Commit message: Added mico_arm to rose's URDF. Actually this would make it rose30 but thats a different topic

File: rose21_urdf/rose21.xacro (robot description, xacro)
@@ -2,4 +2,5 @@
   <xacro:include filename="$(find rose21_urdf)/common.xacro" />
   <xacro:include filename="$(find rose21_urdf)/urdf/wheel_unit_60mm/wheel_unit_60mm_macro.xacro" />
+  <xacro:include filename="$(find mico_description)/urdf/mico_arm.urdf.xacro" />
   <xacro:property name="base_size_x" value="0.76" />
   <xacro:property name="base_size_y" value="0.58" />
@@ -14,4 +15,7 @@
   <xacro:property name="tray_pose_y" value="0.0" />
   <xacro:property name="tray_pose_z" value="0.13" />
+  <xacro:property name="mico_pose_x" value="0.053" />
+  <xacro:property name="mico_pose_y" value="0.17" /> <!-- 5cm from the side of the lift_link -->
+  <xacro:property name="mico_pose_z" value="0.14" />
   <xacro:property name="wheel_front_x"    value="0.28" />
   <xacro:property name="wheel_back_x"     value="-0.305" />
@@ -188,4 +192,6 @@
     <xacro:default_inertial mass="2.0"/>
   </link>
+  <!-- ATTACH ARM -->
+  <xacro:mico_arm parent="lift_link" xyz="${mico_pose_x}  ${mico_pose_y}  ${mico_pose_z}" rpy="0 0 ${pi / 2}"/>
   <!-- START neck -->
   <!-- joint between lift_link and neck_pan -->

Commit message: Removed lift top mimicking

File: rose21_urdf/rose21.xacro (robot description, xacro)
@@ -144,5 +144,4 @@
       <axis xyz="0 1 0" />
       <origin xyz="${-liftsides_size_x} 0 0" rpy="0 0 0"/>
-      <mimic joint="lift_mid_bottom_joint" multiplier="-1"/>
     </joint>
   </xacro:macro>
