Commit message: robot_state_publisher now publishes the kinect frames. In rose_config, kinect.launch should not publish TFs then

File: rose21_urdf/rose21.xacro (robot description, xacro)
@@ -1,2 +1,3 @@
+<?xml version="1.0"?>
 <robot name="Rose20" xmlns:xacro="http://www.ros.org/wiki/xacro">
   <xacro:include filename="$(find rose21_urdf)/common.xacro" />
@@ -232,24 +233,12 @@
   </link>
   <!-- joint between neck_tilt and kinect-->
-  <joint name="kinect_fix" type="fixed">
+<!--   <joint name="kinect_fix" type="fixed">
     <parent link="neck_tilt"/>
     <child link="kinect"/>
     <axis xyz="0 1 0" />
     <origin xyz="${kinect_pose_x} ${kinect_pose_y} ${kinect_pose_z}" rpy="0 0 0"/>
-  </joint>
+  </joint> -->
   <!-- END neck -->
   <!-- START kinect -->
-  <link name='kinect'>
-    <xacro:collission_box   xyz=  "0 0 0.036"
-                            rpy=  "0 0 0"
-                            size= "${kinect_size_x} ${kinect_size_y} ${kinect_size_z}"/>
-    <visual>
-      <origin xyz="0 0 0.036" rpy="0 0 0" />
-        <geometry>
-          <mesh filename="package://rose21_urdf/meshes/kinect.dae"/>
-        </geometry>
-    </visual>
-    <xacro:default_inertial mass="0.1"/>
-  </link>
 <!--   <gazebo reference="kinect">
     <sensor type="depth" name="kinect">
@@ -290,7 +279,8 @@
     <plugin name="NeckController" filename="libNeckController.so"/>
   </gazebo> -->
-  <joint name="link2" type="fixed">
+    <joint name="link2" type="fixed">
       <parent link="neck_tilt"/>
       <child link="camera_center_link"/>
+      <origin xyz="0.03 0 0.07" rpy="0 0 0"/> <!-- Values obtained from neck_tf.cpp-->
     </joint>
     <link name="camera_center_link">
@@ -305,49 +295,5 @@
       </visual>
     </link>
-    <joint name="link3" type="fixed">
-      <parent link="camera_center_link"/>
-      <child link="camera_link"/>
-    </joint>
-    <link name="camera_link">
-      <visual>
-        <origin xyz="0 0 0" rpy="0 0 0" />
-        <geometry>
-          <box size="0.06 0.28 0.04" />
-        </geometry>
-        <material name="black">
-          <color rgba=".1 .1 .1 1" />
-        </material>
-      </visual>
-    </link>
-    <joint name="link4" type="fixed">
-      <parent link="camera_link"/>
-      <child link="camera_rgb_frame"/>
-    </joint>
-    <link name="camera_rgb_frame">
-      <visual>
-        <origin xyz="0 0 0" rpy="0 0 0" />
-        <geometry>
-          <box size="0 0 0" />
-        </geometry>
-        <material name="black">
-          <color rgba=".1 .1 .1 1" />
-        </material>
-      </visual>
-    </link>
-    <joint name="link5" type="fixed">
-      <parent link="camera_rgb_frame"/>
-      <child link="camera_rgb_optical_frame"/>
-    </joint>
-    <link name="camera_rgb_optical_frame">
-      <visual>
-        <origin xyz="0 0 0" rpy="0 0 0" />
-        <geometry>
-          <box size="0 0 0" />
-        </geometry>
-        <material name="black">
-          <color rgba=".1 .1 .1 1" />
-        </material>
-      </visual>
-    </link>
+  <xacro:kinect parent_frame="camera_center_link" xyz="0 0 0" rpy="0 0 0" tf_prefix="rose"/>
     <!-- START Hokuyo -->
   <joint name="hokuyo_joint" type="revolute">

File: rose21_urdf/urdf/kinect/kinect.urdf.xacro (robot description, xacro)
@@ -1,14 +1,24 @@
 <?xml version="1.0"?>
-<robot name="cwru_hardware" xmlns:xacro="http://ros.org/wiki/xacro">
-  <property name="M_PI" value="3.14159"/>
-  <include filename="$(find cwru_description)/urdf/gazebo.urdf.xacro"/>
-<xacro:macro name="kinect" params="xyz rpy parent_frame" >
+<robot xmlns:xi="http://www.w3.org/2001/XInclude"
+    xmlns:gazebo="http://playerstage.sourceforge.net/gazebo/xmlschema/#gz"
+    xmlns:model="http://playerstage.sourceforge.net/gazebo/xmlschema/#model"
+    xmlns:sensor="http://playerstage.sourceforge.net/gazebo/xmlschema/#sensor"
+    xmlns:body="http://playerstage.sourceforge.net/gazebo/xmlschema/#body"
+    xmlns:geom="http://playerstage.sourceforge.net/gazebo/xmlschema/#geom"
+    xmlns:joint="http://playerstage.sourceforge.net/gazebo/xmlschema/#joint"
+    xmlns:controller="http://playerstage.sourceforge.net/gazebo/xmlschema/#controller"
+    xmlns:interface="http://playerstage.sourceforge.net/gazebo/xmlschema/#interface"
+    xmlns:rendering="http://playerstage.sourceforge.net/gazebo/xmlschema/#rendering"
+    xmlns:renderable="http://playerstage.sourceforge.net/gazebo/xmlschema/#renderable"
+    xmlns:physics="http://playerstage.sourceforge.net/gazebo/xmlschema/#physics"
+    xmlns:xacro="http://ros.org/wiki/xacro">
+<xacro:macro name="kinect" params="xyz rpy parent_frame tf_prefix" >
   <joint name="base_camera_joint" type="fixed">
     <origin xyz="${xyz}" rpy="${rpy}" />
     <parent link="${parent_frame}" />
     <origin xyz="0 0 0" rpy="0 0 0" />
-    <child link="camera_link" />
+    <child link="${tf_prefix}/camera_link" />
   </joint>
-  <link name="camera_link">
+  <link name="${tf_prefix}/camera_link">
     <inertial>
       <mass value="0.01" />
@@ -21,5 +31,5 @@
       <origin xyz=" 0 0 0 " rpy="0 0 0" />
       <geometry>
-        <mesh filename="package://cwru_description/meshes/kinect.dae"/>
+        <mesh filename="package://rose21_urdf/meshes/kinect.dae"/>
       </geometry>
     </visual>
@@ -33,8 +43,8 @@
   <joint name="camera_depth_joint" type="fixed">
     <origin xyz="0 0.011 0" rpy="0 0 0" />
-    <parent link="camera_link" />
-    <child link="camera_depth_frame" />
+    <parent link="${tf_prefix}/camera_link" />
+    <child link="${tf_prefix}/camera_depth_frame" />
   </joint>
-  <link name="camera_depth_frame">
+  <link name="${tf_prefix}/camera_depth_frame">
     <inertial>
       <mass value="0.01" />
@@ -47,8 +57,8 @@
   <joint name="camera_depth_optical_joint" type="fixed">
     <origin xyz="0 0 0" rpy="${-M_PI/2} 0 ${-M_PI/2}" />
-    <parent link="camera_depth_frame" />
-    <child link="camera_depth_optical_frame" />
+    <parent link="${tf_prefix}/camera_depth_frame" />
+    <child link="${tf_prefix}/camera_depth_optical_frame" />
   </joint>
-  <link name="camera_depth_optical_frame">
+  <link name="${tf_prefix}/camera_depth_optical_frame">
     <inertial>
       <mass value="0.001" />
@@ -61,8 +71,8 @@
   <joint name="camera_rgb_joint" type="fixed">
     <origin xyz="0 -0.012 0" rpy="0 0 0" />
-    <parent link="camera_link" />
-    <child link="camera_rgb_frame" />
+    <parent link="${tf_prefix}/camera_link" />
+    <child link="${tf_prefix}/camera_rgb_frame" />
   </joint>
-  <link name="camera_rgb_frame">
+  <link name="${tf_prefix}/camera_rgb_frame">
     <inertial>
       <mass value="0.001" />
@@ -75,8 +85,8 @@
   <joint name="camera_rgb_optical_joint" type="fixed">
     <origin xyz="0 0 0" rpy="${-M_PI/2} 0 ${-M_PI/2}" />
-    <parent link="camera_rgb_frame" />
-    <child link="camera_rgb_optical_frame" />
+    <parent link="${tf_prefix}/camera_rgb_frame" />
+    <child link="${tf_prefix}/camera_rgb_optical_frame" />
   </joint>
-  <link name="camera_rgb_optical_frame">
+  <link name="${tf_prefix}/camera_rgb_optical_frame">
     <inertial>
       <mass value="0.001" />
@@ -87,6 +97,4 @@
     </inertial>
   </link>
-  <!-- Kinect sensor for simulation -->
-  <sim_kinect/>
 </xacro:macro>
 </robot>

Commit message: Not prefixing kinect frames.

File: rose21_urdf/rose21.xacro (robot description, xacro)
@@ -294,5 +294,5 @@
       </visual>
     </link>
-  <xacro:kinect parent_frame="camera_center_link" xyz="0 0 0" rpy="0 0 0" tf_prefix="rose"/>
+  <xacro:kinect parent_frame="camera_center_link" xyz="0 0 0" rpy="0 0 0"/>
     <!-- START Hokuyo -->
   <joint name="hokuyo_joint" type="revolute">

File: rose21_urdf/urdf/kinect/kinect.urdf.xacro (robot description, xacro)
@@ -13,12 +13,12 @@
     xmlns:physics="http://playerstage.sourceforge.net/gazebo/xmlschema/#physics"
     xmlns:xacro="http://ros.org/wiki/xacro">
-<xacro:macro name="kinect" params="xyz rpy parent_frame tf_prefix" >
+<xacro:macro name="kinect" params="xyz rpy parent_frame" >
   <joint name="base_camera_joint" type="fixed">
     <origin xyz="${xyz}" rpy="${rpy}" />
     <parent link="${parent_frame}" />
     <origin xyz="0 0 0" rpy="0 0 0" />
-    <child link="${tf_prefix}/camera_link" />
+    <child link="camera_link" />
   </joint>
-  <link name="${tf_prefix}/camera_link">
+  <link name="camera_link">
     <inertial>
       <mass value="0.01" />
@@ -43,8 +43,8 @@
   <joint name="camera_depth_joint" type="fixed">
     <origin xyz="0 0.011 0" rpy="0 0 0" />
-    <parent link="${tf_prefix}/camera_link" />
-    <child link="${tf_prefix}/camera_depth_frame" />
+    <parent link="camera_link" />
+    <child link="camera_depth_frame" />
   </joint>
-  <link name="${tf_prefix}/camera_depth_frame">
+  <link name="camera_depth_frame">
     <inertial>
       <mass value="0.01" />
@@ -57,8 +57,8 @@
   <joint name="camera_depth_optical_joint" type="fixed">
     <origin xyz="0 0 0" rpy="${-M_PI/2} 0 ${-M_PI/2}" />
-    <parent link="${tf_prefix}/camera_depth_frame" />
-    <child link="${tf_prefix}/camera_depth_optical_frame" />
+    <parent link="camera_depth_frame" />
+    <child link="camera_depth_optical_frame" />
   </joint>
-  <link name="${tf_prefix}/camera_depth_optical_frame">
+  <link name="camera_depth_optical_frame">
     <inertial>
       <mass value="0.001" />
@@ -71,8 +71,8 @@
   <joint name="camera_rgb_joint" type="fixed">
     <origin xyz="0 -0.012 0" rpy="0 0 0" />
-    <parent link="${tf_prefix}/camera_link" />
-    <child link="${tf_prefix}/camera_rgb_frame" />
+    <parent link="camera_link" />
+    <child link="camera_rgb_frame" />
   </joint>
-  <link name="${tf_prefix}/camera_rgb_frame">
+  <link name="camera_rgb_frame">
     <inertial>
       <mass value="0.001" />
@@ -85,8 +85,8 @@
   <joint name="camera_rgb_optical_joint" type="fixed">
     <origin xyz="0 0 0" rpy="${-M_PI/2} 0 ${-M_PI/2}" />
-    <parent link="${tf_prefix}/camera_rgb_frame" />
-    <child link="${tf_prefix}/camera_rgb_optical_frame" />
+    <parent link="camera_rgb_frame" />
+    <child link="camera_rgb_optical_frame" />
   </joint>
-  <link name="${tf_prefix}/camera_rgb_optical_frame">
+  <link name="camera_rgb_optical_frame">
     <inertial>
       <mass value="0.001" />

Commit message: Mcio move test

File: rose21_urdf/rose21.xacro (robot description, xacro)
@@ -17,5 +17,5 @@
   <xacro:property name="tray_pose_y" value="0.0" />
   <xacro:property name="tray_pose_z" value="0.13" />
-  <xacro:property name="mico_pose_x" value="0.053" />
+  <xacro:property name="mico_pose_x" value="0.08" />
   <xacro:property name="mico_pose_y" value="0.17" /> <!-- 5cm from the side of the lift_link -->
   <xacro:property name="mico_pose_z" value="0.14" />
@@ -50,4 +50,7 @@
   <xacro:property name="shoulders_size_y" value="0.58" />
   <xacro:property name="shoulders_size_z" value="0.177" />
+  <xacro:property name="shoulders_pose_x" value="0.0" />
+  <xacro:property name="shoulders_pose_y" value="0.0" />
+  <xacro:property name="shoulders_pose_z" value="0.51"/>
   <xacro:property name="lift_rpy" value="0 0 0"/>
   <xacro:property name="neck_tube_size_z" value="0.07" />

Commit message: Added shoulders

File: rose21_urdf/rose21.xacro (robot description, xacro)
@@ -196,4 +196,15 @@
     <xacro:default_inertial mass="2.0"/>
   </link>
+  <joint name="shoulders" type="fixed">
+    <parent link="lift_link"/>
+    <child link="shoulders"/>
+    <origin xyz="0 0 0" rpy="0 0 0"/>
+  </joint>
+  <link name='shoulders'>
+    <xacro:default_box  xyz=  "${shoulders_pose_x} ${shoulders_pose_y} ${shoulders_pose_z}"
+                        rpy=  "0 0 0"
+                        size= "${shoulders_size_x} ${shoulders_size_y} ${shoulders_size_z}"/>
+    <xacro:default_inertial mass="2.0"/>
+  </link>
   <!-- ATTACH ARM -->
   <xacro:mico_arm parent="lift_link" xyz="${mico_pose_x}  ${mico_pose_y}  ${mico_pose_z}" rpy="0 0 ${pi / 2}"/>

Commit message: Added shoulders, fixed neck

File: rose21_urdf/rose21.xacro (robot description, xacro)
@@ -43,5 +43,5 @@
   <xacro:property name="lifttopbox_size_x" value="0.29" />
   <xacro:property name="lifttopbox_size_y" value="0.24" />
-  <xacro:property name="lifttopbox_size_z" value="0.48" /> <!--This excludes the shoulders -->
+  <xacro:property name="lifttopbox_size_z" value="0.52" /> <!--This excludes the shoulders -->
   <xacro:property name="lifttopbox_pose_x" value="-0.10" />
   <xacro:property name="lifttopbox_pose_y" value="0.0" />
@@ -202,5 +202,5 @@
   </joint>
   <link name='shoulders'>
-    <xacro:default_box  xyz=  "${shoulders_pose_x} ${shoulders_pose_y} ${shoulders_pose_z}"
+    <xacro:default_box  xyz=  "${shoulders_pose_x} ${shoulders_pose_y} ${lifttopbox_size_z + shoulders_size_z/2}"
                         rpy=  "0 0 0"
                         size= "${shoulders_size_x} ${shoulders_size_y} ${shoulders_size_z}"/>

Commit message: Added shoulders, fixed neck

File: rose21_urdf/rose21.xacro (robot description, xacro)
@@ -43,5 +43,5 @@
   <xacro:property name="lifttopbox_size_x" value="0.29" />
   <xacro:property name="lifttopbox_size_y" value="0.24" />
-  <xacro:property name="lifttopbox_size_z" value="0.52" /> <!--This excludes the shoulders -->
+  <xacro:property name="lifttopbox_size_z" value="0.48" /> <!--This excludes the shoulders -->
   <xacro:property name="lifttopbox_pose_x" value="-0.10" />
   <xacro:property name="lifttopbox_pose_y" value="0.0" />
@@ -50,7 +50,7 @@
   <xacro:property name="shoulders_size_y" value="0.58" />
   <xacro:property name="shoulders_size_z" value="0.177" />
-  <xacro:property name="shoulders_pose_x" value="0.0" />
+  <xacro:property name="shoulders_pose_x" value="-0.10" />
   <xacro:property name="shoulders_pose_y" value="0.0" />
-  <xacro:property name="shoulders_pose_z" value="0.51"/>
+  <xacro:property name="shoulders_pose_z" value="0.0"/>
   <xacro:property name="lift_rpy" value="0 0 0"/>
   <xacro:property name="neck_tube_size_z" value="0.07" />

Commit message: Added shoulders, fixed neck

File: rose21_urdf/rose21.xacro (robot description, xacro)
@@ -47,8 +47,8 @@
   <xacro:property name="lifttopbox_pose_y" value="0.0" />
   <xacro:property name="lifttopbox_pose_z" value="0.285"/>
-  <xacro:property name="shoulders_size_x" value="0.265" />
+  <xacro:property name="shoulders_size_x" value="0.21" />
   <xacro:property name="shoulders_size_y" value="0.58" />
   <xacro:property name="shoulders_size_z" value="0.177" />
-  <xacro:property name="shoulders_pose_x" value="-0.10" />
+  <xacro:property name="shoulders_pose_x" value="-0.08" />
   <xacro:property name="shoulders_pose_y" value="0.0" />
   <xacro:property name="shoulders_pose_z" value="0.0"/>

Commit message: Fixed lift_mid height

File: rose21_urdf/rose21.xacro (robot description, xacro)
@@ -10,5 +10,5 @@
   <xacro:property name="base_pose_x" value="0.0" />
   <xacro:property name="base_pose_y" value="0.0" />
-  <xacro:property name="base_pose_z" value="0.20" />
+  <xacro:property name="base_pose_z" value="0.26" />
   <xacro:property name="tray_size_x" value="0.20" />
   <xacro:property name="tray_size_y" value="0.20" />

Commit message: Fixed base size

File: rose21_urdf/rose21.xacro (robot description, xacro)
@@ -7,5 +7,5 @@
   <xacro:property name="base_size_x" value="0.76" />
   <xacro:property name="base_size_y" value="0.58" />
-  <xacro:property name="base_size_z" value="0.05" />
+  <xacro:property name="base_size_z" value="0.12" />
   <xacro:property name="base_pose_x" value="0.0" />
   <xacro:property name="base_pose_y" value="0.0" />

Commit message: Fixed tray size

File: rose21_urdf/rose21.xacro (robot description, xacro)
@@ -16,5 +16,5 @@
   <xacro:property name="tray_pose_x" value="0.135" />
   <xacro:property name="tray_pose_y" value="0.0" />
-  <xacro:property name="tray_pose_z" value="0.13" />
+  <xacro:property name="tray_pose_z" value="0.10" />
   <xacro:property name="mico_pose_x" value="0.08" />
   <xacro:property name="mico_pose_y" value="0.17" /> <!-- 5cm from the side of the lift_link -->

Commit message: Fixed neck pose

File: rose21_urdf/rose21.xacro (robot description, xacro)
@@ -59,5 +59,5 @@
   <xacro:property name="neck_pan_size_y" value="0.04" />
   <xacro:property name="neck_pan_size_z" value="0.02" />
-  <xacro:property name="neck_pan_pose_x" value="0.015" />
+  <xacro:property name="neck_pan_pose_x" value="0.075" /> <!--relative to lift_link -->
   <xacro:property name="neck_pan_pose_y" value="0.00" />
   <xacro:property name="neck_pan_pose_z" value="0.00" />
@@ -224,5 +224,5 @@
    -->
   <link name='neck_pan'>
-    <xacro:default_box  xyz=  "${neck_pan_size_x/2} 0 ${neck_pan_size_z/2 + neck_tube_size_z}"
+    <xacro:default_box  xyz=  "${neck_pan_pose_x} 0 ${neck_pan_size_z/2 + neck_tube_size_z}"
                         rpy=  "0 0 0"
                         size= "${neck_pan_size_x} ${neck_pan_size_y} ${neck_pan_size_z}"/>

Commit message: Fixed neck pose

File: rose21_urdf/rose21.xacro (robot description, xacro)
@@ -59,5 +59,5 @@
   <xacro:property name="neck_pan_size_y" value="0.04" />
   <xacro:property name="neck_pan_size_z" value="0.02" />
-  <xacro:property name="neck_pan_pose_x" value="0.075" /> <!--relative to lift_link -->
+  <xacro:property name="neck_pan_pose_x" value="0.08" /> <!--relative to lift_link -->
   <xacro:property name="neck_pan_pose_y" value="0.00" />
   <xacro:property name="neck_pan_pose_z" value="0.00" />

Commit message: Fixed neck pose

File: rose21_urdf/rose21.xacro (robot description, xacro)
@@ -59,5 +59,5 @@
   <xacro:property name="neck_pan_size_y" value="0.04" />
   <xacro:property name="neck_pan_size_z" value="0.02" />
-  <xacro:property name="neck_pan_pose_x" value="0.08" /> <!--relative to lift_link -->
+  <xacro:property name="neck_pan_pose_x" value="-0.08" /> <!--relative to lift_link -->
   <xacro:property name="neck_pan_pose_y" value="0.00" />
   <xacro:property name="neck_pan_pose_z" value="0.00" />

Commit message: Fixed neck pose

File: rose21_urdf/rose21.xacro (robot description, xacro)
@@ -215,5 +215,5 @@
     <child link="neck_pan"/>
     <axis xyz="0 0 1" />
-    <origin xyz="${lifttopbox_pose_x} 0 ${lifttopbox_size_z + shoulders_size_z}" rpy="0 0 0"/>
+    <origin xyz="${neck_pan_pose_x} 0 ${lifttopbox_size_z + shoulders_size_z}" rpy="0 0 0"/>
     <dynamics damping="1.0" friction="1.0"/>
     <limit effort="1.0" lower="-0.7853" upper="0.7853" velocity="10.0"/>
@@ -224,5 +224,5 @@
    -->
   <link name='neck_pan'>
-    <xacro:default_box  xyz=  "${neck_pan_pose_x} 0 ${neck_pan_size_z/2 + neck_tube_size_z}"
+    <xacro:default_box  xyz=  "${neck_pan_size_x/2} 0 ${neck_pan_size_z/2 + neck_tube_size_z}"
                         rpy=  "0 0 0"
                         size= "${neck_pan_size_x} ${neck_pan_size_y} ${neck_pan_size_z}"/>

Commit message: Fixed lifttopboxpose

File: rose21_urdf/rose21.xacro (robot description, xacro)
@@ -44,5 +44,5 @@
   <xacro:property name="lifttopbox_size_y" value="0.24" />
   <xacro:property name="lifttopbox_size_z" value="0.48" /> <!--This excludes the shoulders -->
-  <xacro:property name="lifttopbox_pose_x" value="-0.10" />
+  <xacro:property name="lifttopbox_pose_x" value="-0.115" />
   <xacro:property name="lifttopbox_pose_y" value="0.0" />
   <xacro:property name="lifttopbox_pose_z" value="0.285"/>

Commit message: Fixed neck tf

File: rose21_urdf/rose21.xacro (robot description, xacro)
@@ -54,5 +54,5 @@
   <xacro:property name="shoulders_pose_z" value="0.0"/>
   <xacro:property name="lift_rpy" value="0 0 0"/>
-  <xacro:property name="neck_tube_size_z" value="0.07" />
+  <xacro:property name="neck_tube_size_z" value="0.06" />
   <xacro:property name="neck_tube_diameter" value="0.03" />
   <xacro:property name="neck_pan_size_x" value="0.298" />
@@ -66,5 +66,5 @@
   <xacro:property name="neck_tilt_size_z" value="0.048" />
   <xacro:property name="neck_tilt_servo_center_z" value="0.033" />
-  <xacro:property name="neck_tilt_pose_x" value="0.28" /> <!--Distance between tilt axis and neck pan tube -->
+  <xacro:property name="neck_tilt_pose_x" value="0.284" /> <!--Distance between tilt axis and neck pan tube -->
   <xacro:property name="neck_tilt_pose_y" value="0.00" />
   <xacro:property name="neck_tilt_pose_z" value="0.115" /> <!--Height of the tilt axis from top of shoulders-->

Commit message: Fixed arm location

File: rose21_urdf/rose21.xacro (robot description, xacro)
@@ -17,7 +17,7 @@
   <xacro:property name="tray_pose_y" value="0.0" />
   <xacro:property name="tray_pose_z" value="0.10" />
-  <xacro:property name="mico_pose_x" value="0.08" />
-  <xacro:property name="mico_pose_y" value="0.17" /> <!-- 5cm from the side of the lift_link -->
-  <xacro:property name="mico_pose_z" value="0.14" />
+  <xacro:property name="mico_pose_x" value="0.114" />
+  <xacro:property name="mico_pose_y" value="0.197" /> <!-- 5cm from the side of the lift_link -->
+  <xacro:property name="mico_pose_z" value="0.094" />
   <xacro:property name="wheel_front_x"    value="0.28" />
   <xacro:property name="wheel_back_x"     value="-0.305" />

Commit message: Do not include mico in robot model, this is done sperately for now.

File: rose21_urdf/rose21.xacro (robot description, xacro)
@@ -3,5 +3,5 @@
   <xacro:include filename="$(find rose21_urdf)/common.xacro" />
   <xacro:include filename="$(find opteq_wheelunits_01)/urdf/wheel_unit_60mm_macro.xacro" />
-  <xacro:include filename="$(find mico_description)/urdf/mico_arm.urdf.xacro" />
+  <!-- <xacro:include filename="$(find mico_description)/urdf/mico_arm.urdf.xacro" /> -->
   <xacro:include filename="$(find kinect_description)/urdf/kinect.urdf.xacro" />
   <xacro:property name="base_size_x" value="0.76" />
@@ -208,5 +208,10 @@
   </link>
   <!-- ATTACH ARM -->
-  <xacro:mico_arm parent="lift_link" xyz="${mico_pose_x}  ${mico_pose_y}  ${mico_pose_z}" rpy="0 0 ${pi / 2}"/>
+  <!-- <xacro:mico_arm parent="lift_link" xyz="${mico_pose_x}  ${mico_pose_y}  ${mico_pose_z}" rpy="0 0 ${pi / 2}"/> -->
+  <joint name="mico_root_mount_joint" type="fixed">
+    <parent link="lift_link"/>
+    <child link="mico_root"/>
+    <origin xyz="${mico_pose_x}  ${mico_pose_y}  ${mico_pose_z}" rpy="0 0 ${pi / 2}"/>
+  </joint>
   <!-- START neck -->
   <!-- joint between lift_link and neck_pan -->
